Commit message: rotating the kinect so that it's horizontal, otherwise point cloud is not placed correctly - bug in simulated kinect?

File: sr_description/other/xacro/kinect/gazebo_kinect.urdf.xacro (robot description, xacro)
@@ -2,5 +2,5 @@
 <xacro:macro name="shadowarm_sim_kinect">
   <gazebo reference="camera_link">
-    <sensor:camera name="kinect_camera">
+    <sensor:camera name="camera">
       <imageFormat>R8G8B8</imageFormat>
       <imageSize>640 480</imageSize>
@@ -11,18 +11,24 @@
       <baseline>0.1</baseline>
       <controller:gazebo_ros_openni_kinect name="kinect_camera_controller" plugin="libgazebo_ros_openni_kinect.so">
+        <cameraName>kinect</cameraName>
         <alwaysOn>true</alwaysOn>
         <updateRate>20</updateRate>
         <imageTopicName>/camera/image_raw</imageTopicName>
-	<pointCloudTopicName>/camera/depth_registered/points</pointCloudTopicName>
+        <pointCloudTopicName>/camera/depth_registered/points</pointCloudTopicName>
         <cameraInfoTopicName>/camera/camera_info</cameraInfoTopicName>
-        <frameName>/camera_depth_optical_frame</frameName>
-        <distortion_k1>0.0</distortion_k1>
-        <distortion_k2>0.0</distortion_k2>
-        <distortion_k3>0.0</distortion_k3>
-        <distortion_t1>0.0</distortion_t1>
-        <distortion_t2>0.0</distortion_t2>
+        <frameName>camera_depth_optical_frame</frameName>
+        <CxPrime>0.0</CxPrime>
+        <Cx>0.0</Cx>
+        <Cy>0.0</Cy>
+        <focalLength>0.0</focalLength>
+        <hackBaseline>0.0</hackBaseline>
+        <distortionK1>0.0</distortionK1>
+        <distortionK2>0.0</distortionK2>
+        <distortionK3>0.0</distortionK3>
+        <distortionT1>0.0</distortionT1>
+        <distortionT2>0.0</distortionT2>
       </controller:gazebo_ros_openni_kinect>
     </sensor:camera>
   </gazebo>
-</xacro:macro>
+  </xacro:macro>
 </robot>

File: sr_description/other/xacro/kinect/shadowarm_kinect.urdf.xacro (robot description, xacro)
@@ -6,6 +6,6 @@
       <!--	  <origin xyz="0.00724 0.153 0.4405"
 	  rpy="-${M_PI/2} 0.5236 -0.2618" /> -->
-      <origin xyz="0.01216 0.1713 0.433"
-	      rpy="-${M_PI/2} ${M_PI/4} -${M_PI/12}" />
+      <origin  xyz="0.01216 0.1713 0.433"
+	       rpy="0 ${M_PI/4} -${M_PI/12}" />
       <parent link="${parent}"/>
       <child link="camera_link" />
@@ -88,5 +88,4 @@
       </inertial>
     </link>
-    <!-- Kinect sensor for simulation -->
     <shadowarm_sim_kinect/>
   </xacro:macro>
