Commit message: kinect model modified, the point cloud is now properly published

File: sr_description/other/xacro/kinect/shadowarm_kinect.urdf.xacro (robot description, xacro)
@@ -6,6 +6,6 @@
       <!--	  <origin xyz="0.00724 0.153 0.4405"
 	  rpy="-${M_PI/2} 0.5236 -0.2618" /> -->
-      <origin xyz="0.01216 0.1713 0.433"
-	      rpy="-${M_PI/2} ${M_PI/4} -${M_PI/12}" />
+      <origin xyz="0 0 0"
+	      rpy="0 0 0" />
       <parent link="${parent}"/>
       <child link="camera_link" />
@@ -26,5 +26,6 @@
       </visual>
       <collision>
-	<origin xyz="0.0 0.0 0.0" rpy="0 0 0" />
+	<origin xyz="-0.02434 0.1713 0.433"
+              rpy="-${M_PI/2} ${M_PI/4} -${M_PI/12}"/>
 	<geometry>
 	  <box size="0.0730 .2760 0.0720"/>
