Commit message: fixed wrist

File: sr_description/hand/xacro/palm/palm.urdf.xacro (robot description, xacro)
@@ -46,5 +46,5 @@
       </collision>
     </link>
-    <joint name="${prefix}WRJ1" type="revolute">
+    <joint name="${prefix}WRJ1" type="fixed">
       <parent link="${parent}"/>
       <child link="${prefix}palm"/>

File: sr_description/hand/xacro/wrist/wrist.urdf.xacro (robot description, xacro)
@@ -55,5 +55,5 @@
       <selfCollide>false</selfCollide>
     </gazebo>
-    <joint name="${prefix}WRJ2" type="revolute">
+    <joint name="${prefix}WRJ2" type="fixed">
       <parent link="${parent}"/>
       <child link="${prefix}wrist"/>
