Commit message: Simple joints are working in Gazebo

File: sr_description/hand/xacro/finger/knuckle/knuckle.transmission.xacro (robot description, xacro)
@@ -9,18 +9,22 @@
   <!-- joint_prefix prepends fingername to the joint names -->
   <xacro:macro name="knuckle_transmission" params="muscletrans prefix joint_prefix link_prefix" >
-   <!-- muscle hand -->
+    <!-- muscle hand -->
     <xacro:if value="${muscletrans}">
       <transmission type="sr_mechanism_model/SimpleTransmissionForMuscle" name="${prefix}${link_prefix}knuckle_transmission">
-      <actuator name="${prefix}${joint_prefix}J4" />
-      <joint name="${prefix}${joint_prefix}J4" />
-      <mechanicalReduction>1</mechanicalReduction>
+        <actuator name="${prefix}${joint_prefix}J4" />
+        <joint name="${prefix}${joint_prefix}J4" />
+        <mechanicalReduction>1</mechanicalReduction>
       </transmission>
     </xacro:if>
     <!-- motor hand -->
     <xacro:unless value="${muscletrans}">
-      <transmission type="transmission_interface/SimpleTransmission" name="${prefix}${link_prefix}knuckle_transmission">
-      <actuator name="${prefix}${joint_prefix}J4" />
-      <joint name="${prefix}${joint_prefix}J4" />
-      <mechanicalReduction>1</mechanicalReduction>
+      <transmission name="${prefix}${link_prefix}knuckle_transmission">
+        <type>transmission_interface/SimpleTransmission</type>
+        <actuator name="${prefix}${joint_prefix}J4">
+          <mechanicalReduction>1</mechanicalReduction>
+        </actuator>
+        <joint name="${prefix}${joint_prefix}J4">
+          <hardwareInterface>EffortJointInterface</hardwareInterface>
+        </joint>
       </transmission>
     </xacro:unless>

File: sr_description/hand/xacro/finger/lfmetacarpal/lfmetacarpal.transmission.xacro (robot description, xacro)
@@ -7,18 +7,22 @@
   <!-- prefix can be anything but usually is "r_" or  "l_" for right and left hands distinction -->
   <xacro:macro name="lfmetacarpal_transmission" params="muscletrans prefix" >
-   <!-- muscle hand -->
+    <!-- muscle hand -->
     <xacro:if value="${muscletrans}">
       <transmission type="sr_mechanism_model/SimpleTransmissionForMuscle" name="${prefix}lfmetacarpal_transmission">
-      <actuator name="${prefix}LFJ5" />
-      <joint name="${prefix}LFJ5" />
-      <mechanicalReduction>1</mechanicalReduction>
+        <actuator name="${prefix}LFJ5" />
+        <joint name="${prefix}LFJ5" />
+        <mechanicalReduction>1</mechanicalReduction>
       </transmission>
     </xacro:if>
     <!-- motor hand -->
     <xacro:unless value="${muscletrans}">
-      <transmission type="transmission_interface/SimpleTransmission" name="${prefix}lfmetacarpal_transmission">
-      <actuator name="${prefix}LFJ5" />
-      <joint name="${prefix}LFJ5" />
-      <mechanicalReduction>1</mechanicalReduction>
+      <transmission name="${prefix}lfmetacarpal_transmission">
+        <type>transmission_interface/SimpleTransmission</type>
+        <actuator name="${prefix}LFJ5">
+          <mechanicalReduction>1</mechanicalReduction>
+        </actuator>
+        <joint name="${prefix}LFJ5">
+          <hardwareInterface>EffortJointInterface</hardwareInterface>
+        </joint>
       </transmission>
     </xacro:unless>

File: sr_description/hand/xacro/finger/middle/middle.transmission.xacro (robot description, xacro)
@@ -9,20 +9,26 @@
   <!-- joint_prefix prepends fingername to the joint names -->
   <xacro:macro name="middle_transmission" params="muscletrans prefix joint_prefix link_prefix" >
-   <!-- muscle hand -->
+    <!-- muscle hand -->
     <xacro:if value="${muscletrans}">
       <transmission type="sr_mechanism_model/J0TransmissionForMuscle" name="${prefix}${link_prefix}middle_transmission">
-      <actuator name="${prefix}${joint_prefix}J0" />
-      <joint name="${prefix}${joint_prefix}J1" />
-      <joint name="${prefix}${joint_prefix}J2" />
-      <mechanicalReduction>1</mechanicalReduction>
+        <actuator name="${prefix}${joint_prefix}J0" />
+        <joint name="${prefix}${joint_prefix}J1" />
+        <joint name="${prefix}${joint_prefix}J2" />
+        <mechanicalReduction>1</mechanicalReduction>
       </transmission>
     </xacro:if>
     <!-- motor hand -->
     <xacro:unless value="${muscletrans}">
-      <transmission type="transmission_interface/SimpleTransmission" name="${prefix}${link_prefix}middle_transmission">
-      <actuator name="${prefix}${joint_prefix}J0" />
-      <joint name="${prefix}${joint_prefix}J1" />
-      <joint name="${prefix}${joint_prefix}J2" />
-      <mechanicalReduction>1</mechanicalReduction>
+      <transmission name="${prefix}${link_prefix}middle_transmission">
+        <type>transmission_interface/SimpleTransmission</type>
+        <actuator name="${prefix}${joint_prefix}J0">
+          <mechanicalReduction>1</mechanicalReduction>
+        </actuator>
+        <joint name="${prefix}${joint_prefix}J1">
+          <hardwareInterface>EffortJointInterface</hardwareInterface>
+        </joint>
+        <!--<joint name="${prefix}${joint_prefix}J2">-->
+          <!--<hardwareInterface>EffortJointInterface</hardwareInterface>-->
+        <!--</joint>-->
       </transmission>
     </xacro:unless>

File: sr_description/hand/xacro/finger/proximal/proximal.transmission.xacro (robot description, xacro)
@@ -9,18 +9,22 @@
   <!-- joint_prefix prepends fingername to the joint names -->
   <xacro:macro name="proximal_transmission" params="muscletrans prefix joint_prefix link_prefix" >
-   <!-- muscle hand -->
+    <!-- muscle hand -->
     <xacro:if value="${muscletrans}">
       <transmission type="sr_mechanism_model/SimpleTransmissionForMuscle" name="${prefix}${link_prefix}proximal_transmission">
-      <actuator name="${prefix}${joint_prefix}J3" />
-      <joint name="${prefix}${joint_prefix}J3" />
-      <mechanicalReduction>1</mechanicalReduction>
+        <actuator name="${prefix}${joint_prefix}J3" />
+        <joint name="${prefix}${joint_prefix}J3" />
+        <mechanicalReduction>1</mechanicalReduction>
       </transmission>
     </xacro:if>
     <!-- motor hand -->
     <xacro:unless value="${muscletrans}">
-      <transmission type="transmission_interface/SimpleTransmission" name="${prefix}${link_prefix}proximal_transmission">
-      <actuator name="${prefix}${joint_prefix}J3" />
-      <joint name="${prefix}${joint_prefix}J3" />
-      <mechanicalReduction>1</mechanicalReduction>
+      <transmission name="${prefix}${link_prefix}proximal_transmission">
+        <type>transmission_interface/SimpleTransmission</type>
+        <actuator name="${prefix}${joint_prefix}J3">
+          <mechanicalReduction>1</mechanicalReduction>
+        </actuator>
+        <joint name="${prefix}${joint_prefix}J3">
+          <hardwareInterface>EffortJointInterface</hardwareInterface>
+        </joint>
       </transmission>
     </xacro:unless>

File: sr_description/hand/xacro/palm/palm.transmission.xacro (robot description, xacro)
@@ -7,18 +7,22 @@
   <!-- prefix can be anything but usually is "r_" or  "l_" for right and left hands distinction -->
   <xacro:macro name="shadowhand_palm_transmission" params="muscletrans prefix" >
-   <!-- muscle hand -->
+    <!-- muscle hand -->
     <xacro:if value="${muscletrans}">
       <transmission type="sr_mechanism_model/SimpleTransmissionForMuscle" name="${prefix}palm_transmission">
-      <actuator name="${prefix}WRJ1" />
-      <joint name="${prefix}WRJ1" />
-      <mechanicalReduction>1</mechanicalReduction>
+        <actuator name="${prefix}WRJ1" />
+        <joint name="${prefix}WRJ1" />
+        <mechanicalReduction>1</mechanicalReduction>
       </transmission>
     </xacro:if>
     <!-- motor hand -->
     <xacro:unless value="${muscletrans}">
-      <transmission type="transmission_interface/SimpleTransmission" name="${prefix}palm_transmission">
-      <actuator name="${prefix}WRJ1" />
-      <joint name="${prefix}WRJ1" />
-      <mechanicalReduction>1</mechanicalReduction>
+      <transmission name="${prefix}palm_transmission">
+        <type>transmission_interface/SimpleTransmission</type>
+        <actuator name="${prefix}WRJ1">
+          <mechanicalReduction>1</mechanicalReduction>
+        </actuator>
+        <joint name="${prefix}WRJ1">
+          <hardwareInterface>EffortJointInterface</hardwareInterface>
+        </joint>
       </transmission>
     </xacro:unless>

File: sr_description/hand/xacro/thumb/thbase.transmission.xacro (robot description, xacro)
@@ -7,18 +7,22 @@
   <!-- prefix can be anything but usually is "r_" or  "l_" for right and left hands distinction -->
   <xacro:macro name="thbase_transmission" params="muscletrans prefix" >
-   <!-- muscle hand -->
+    <!-- muscle hand -->
     <xacro:if value="${muscletrans}">
       <transmission type="sr_mechanism_model/SimpleTransmissionForMuscle" name="${prefix}thbase_transmission">
-      <actuator name="${prefix}THJ5" />
-      <joint name="${prefix}THJ5" />
-      <mechanicalReduction>1</mechanicalReduction>
+        <actuator name="${prefix}THJ5" />
+        <joint name="${prefix}THJ5" />
+        <mechanicalReduction>1</mechanicalReduction>
       </transmission>
     </xacro:if>
     <!-- motor hand -->
     <xacro:unless value="${muscletrans}">
-      <transmission type="transmission_interface/SimpleTransmission" name="${prefix}thbase_transmission">
-      <actuator name="${prefix}THJ5" />
-      <joint name="${prefix}THJ5" />
-      <mechanicalReduction>1</mechanicalReduction>
+      <transmission name="${prefix}thbase_transmission">
+        <type>transmission_interface/SimpleTransmission</type>
+        <actuator name="${prefix}THJ5">
+          <mechanicalReduction>1</mechanicalReduction>
+        </actuator>
+        <joint name="${prefix}THJ5">
+          <hardwareInterface>EffortJointInterface</hardwareInterface>
+        </joint>
       </transmission>
     </xacro:unless>

File: sr_description/hand/xacro/thumb/thdistal.transmission.xacro (robot description, xacro)
@@ -7,20 +7,24 @@
   <!-- prefix can be anything but usually is "r_" or  "l_" for right and left hands distinction -->
   <xacro:macro name="thdistal_transmission" params="muscletrans prefix" >
-   <!-- muscle hand -->
+    <!-- muscle hand -->
     <xacro:if value="${muscletrans}">
       <transmission type="sr_mechanism_model/SimpleTransmissionForMuscle" name="${prefix}thdistal_transmission">
-      <actuator name="${prefix}THJ1" />
-      <joint name="${prefix}THJ1" />
-      <mechanicalReduction>1</mechanicalReduction>
+        <actuator name="${prefix}THJ1" />
+        <joint name="${prefix}THJ1" />
+        <mechanicalReduction>1</mechanicalReduction>
       </transmission>
     </xacro:if>
     <!-- motor hand -->
     <xacro:unless value="${muscletrans}">
-      <transmission type="transmission_interface/SimpleTransmission" name="${prefix}thdistal_transmission">
-      <actuator name="${prefix}THJ1" />
-      <joint name="${prefix}THJ1" />
-      <mechanicalReduction>1</mechanicalReduction>
+      <transmission name="${prefix}thdistal_transmission">
+        <type>transmission_interface/SimpleTransmission</type>
+        <actuator name="${prefix}THJ1">
+          <mechanicalReduction>1</mechanicalReduction>
+        </actuator>
+        <joint name="${prefix}THJ1">
+          <hardwareInterface>EffortJointInterface</hardwareInterface>
+        </joint>
       </transmission>
     </xacro:unless>
   </xacro:macro>
-  </robot>
+</robot>

File: sr_description/hand/xacro/thumb/thhub.transmission.xacro (robot description, xacro)
@@ -7,18 +7,22 @@
   <!-- prefix can be anything but usually is "r_" or  "l_" for right and left hands distinction -->
   <xacro:macro name="thhub_transmission" params="muscletrans prefix" >
-   <!-- muscle hand -->
+    <!-- muscle hand -->
     <xacro:if value="${muscletrans}">
       <transmission type="sr_mechanism_model/SimpleTransmissionForMuscle" name="${prefix}thhub_transmission">
-      <actuator name="${prefix}THJ3" />
-      <joint name="${prefix}THJ3" />
-      <mechanicalReduction>1</mechanicalReduction>
+        <actuator name="${prefix}THJ3" />
+        <joint name="${prefix}THJ3" />
+        <mechanicalReduction>1</mechanicalReduction>
       </transmission>
     </xacro:if>
     <!-- motor hand -->
     <xacro:unless value="${muscletrans}">
-      <transmission type="transmission_interface/SimpleTransmission" name="${prefix}thhub_transmission">
-      <actuator name="${prefix}THJ3" />
-      <joint name="${prefix}THJ3" />
-      <mechanicalReduction>1</mechanicalReduction>
+      <transmission name="${prefix}thhub_transmission">
+        <type>transmission_interface/SimpleTransmission</type>
+        <actuator name="${prefix}THJ3">
+          <mechanicalReduction>1</mechanicalReduction>
+        </actuator>
+        <joint name="${prefix}THJ3">
+          <hardwareInterface>EffortJointInterface</hardwareInterface>
+        </joint>
       </transmission>
     </xacro:unless>

File: sr_description/hand/xacro/thumb/thmiddle.transmission.xacro (robot description, xacro)
@@ -7,18 +7,22 @@
   <!-- prefix can be anything but usually is "r_" or  "l_" for right and left hands distinction -->
   <xacro:macro name="thmiddle_transmission" params="muscletrans prefix" >
-   <!-- muscle hand -->
+    <!-- muscle hand -->
     <xacro:if value="${muscletrans}">
       <transmission type="sr_mechanism_model/SimpleTransmissionForMuscle" name="${prefix}thmiddle_transmission">
-      <actuator name="${prefix}THJ2" />
-      <joint name="${prefix}THJ2" />
-      <mechanicalReduction>1</mechanicalReduction>
+        <actuator name="${prefix}THJ2" />
+        <joint name="${prefix}THJ2" />
+        <mechanicalReduction>1</mechanicalReduction>
       </transmission>
     </xacro:if>
     <!-- motor hand -->
     <xacro:unless value="${muscletrans}">
-      <transmission type="transmission_interface/SimpleTransmission" name="${prefix}thmiddle_transmission">
-      <actuator name="${prefix}THJ2" />
-      <joint name="${prefix}THJ2" />
-      <mechanicalReduction>1</mechanicalReduction>
+      <transmission name="${prefix}thmiddle_transmission">
+        <type>transmission_interface/SimpleTransmission</type>
+        <actuator name="${prefix}THJ2">
+          <mechanicalReduction>1</mechanicalReduction>
+        </actuator>
+        <joint name="${prefix}THJ2">
+          <hardwareInterface>EffortJointInterface</hardwareInterface>
+        </joint>
       </transmission>
     </xacro:unless>

File: sr_description/hand/xacro/thumb/thproximal.transmission.xacro (robot description, xacro)
@@ -7,18 +7,22 @@
   <!-- prefix can be anything but usually is "r_" or  "l_" for right and left hands distinction -->
   <xacro:macro name="thproximal_transmission" params="muscletrans prefix" >
-   <!-- muscle hand -->
+    <!-- muscle hand -->
     <xacro:if value="${muscletrans}">
       <transmission type="sr_mechanism_model/SimpleTransmissionForMuscle" name="${prefix}thproximal_transmission">
-      <actuator name="${prefix}THJ4" />
-      <joint name="${prefix}THJ4" />
-      <mechanicalReduction>1</mechanicalReduction>
+        <actuator name="${prefix}THJ4" />
+        <joint name="${prefix}THJ4" />
+        <mechanicalReduction>1</mechanicalReduction>
       </transmission>
     </xacro:if>
     <!-- motor hand -->
     <xacro:unless value="${muscletrans}">
-      <transmission type="transmission_interface/SimpleTransmission" name="${prefix}thproximal_transmission">
-      <actuator name="${prefix}THJ4" />
-      <joint name="${prefix}THJ4" />
-      <mechanicalReduction>1</mechanicalReduction>
+      <transmission name="${prefix}thproximal_transmission">
+        <type>transmission_interface/SimpleTransmission</type>
+        <actuator name="${prefix}THJ4">
+          <mechanicalReduction>1</mechanicalReduction>
+        </actuator>
+        <joint name="${prefix}THJ4">
+          <hardwareInterface>EffortJointInterface</hardwareInterface>
+        </joint>
       </transmission>
     </xacro:unless>

File: sr_description/hand/xacro/wrist/wrist.transmission.xacro (robot description, xacro)
@@ -17,8 +17,12 @@
     <!-- motor hand -->
     <xacro:unless value="${muscletrans}">
-      <transmission type="transmission_interface/SimpleTransmission" name="${prefix}wrist_transmission">
-        <actuator name="${prefix}WRJ2" />
-        <joint name="${prefix}WRJ2" />
-        <mechanicalReduction>1</mechanicalReduction>
+      <transmission name="${prefix}wrist_transmission">
+        <type>transmission_interface/SimpleTransmission</type>
+        <actuator name="${prefix}WRJ2">
+          <mechanicalReduction>1</mechanicalReduction>
+        </actuator>
+        <joint name="${prefix}WRJ2">
+          <hardwareInterface>EffortJointInterface</hardwareInterface>
+        </joint>
       </transmission>
     </xacro:unless>

File: sr_description/other/xacro/gazebo/gazebo.urdf.xacro (robot description, xacro)
@@ -3,9 +3,17 @@
 xmlns:controller="http://playerstage.sourceforge.net/gazebo/xmlschema/#controller"
 xmlns:interface="http://playerstage.sourceforge.net/gazebo/xmlschema/#interface">
+  <!--<gazebo>-->
+    <!--<plugin name="sr_gazebo_ros_controller_manager"-->
+    <!--filename="libsr_gazebo_ros_controller_manager.so">-->
+      <!--<alwaysOn>true</alwaysOn>-->
+      <!--<updateRate>1400.0</updateRate>-->
+      <!--&lt;!&ndash; <robotParam>sh_description</robotParam> &ndash;&gt;-->
+    <!--</plugin>-->
+  <!--</gazebo>-->
   <gazebo>
-    <plugin name="sr_gazebo_ros_controller_manager"
-    filename="libsr_gazebo_ros_controller_manager.so">
-      <alwaysOn>true</alwaysOn>
-      <updateRate>1400.0</updateRate>
+    <plugin name="gazebo_ros_control" filename="libgazebo_ros_control.so">
+       <!--<robotNamespace>/shadowhand_motor</robotNamespace>-->
+      <!--<alwaysOn>true</alwaysOn>-->
+      <!--<updateRate>1400.0</updateRate>-->
       <!-- <robotParam>sh_description</robotParam> -->
     </plugin>
