Commit message: Reverted controllers for Shadow's and adding ros control plugin instead of Shadow's

File: sr_description/hand/xacro/finger/middle/middle.transmission.xacro (robot description, xacro)
@@ -21,5 +21,5 @@
     <xacro:unless value="${muscletrans}">
       <transmission name="${prefix}${link_prefix}middle_transmission">
-        <type>transmission_interface/SimpleTransmission</type>
+        <type>sr_mechanism_model/J0Transmission</type>
         <actuator name="${prefix}${joint_prefix}J0">
           <mechanicalReduction>1</mechanicalReduction>
@@ -27,8 +27,6 @@
         <joint name="${prefix}${joint_prefix}J1">
           <hardwareInterface>EffortJointInterface</hardwareInterface>
+          <dependentJoint name="${prefix}${joint_prefix}J2"/>
         </joint>
-        <!--<joint name="${prefix}${joint_prefix}J2">-->
-          <!--<hardwareInterface>EffortJointInterface</hardwareInterface>-->
-        <!--</joint>-->
       </transmission>
     </xacro:unless>

File: sr_description/other/xacro/gazebo/gazebo.urdf.xacro (robot description, xacro)
@@ -3,18 +3,8 @@
 xmlns:controller="http://playerstage.sourceforge.net/gazebo/xmlschema/#controller"
 xmlns:interface="http://playerstage.sourceforge.net/gazebo/xmlschema/#interface">
-  <!--<gazebo>-->
-    <!--<plugin name="sr_gazebo_ros_controller_manager"-->
-    <!--filename="libsr_gazebo_ros_controller_manager.so">-->
-      <!--<alwaysOn>true</alwaysOn>-->
-      <!--<updateRate>1400.0</updateRate>-->
-      <!--&lt;!&ndash; <robotParam>sh_description</robotParam> &ndash;&gt;-->
-    <!--</plugin>-->
-  <!--</gazebo>-->
   <gazebo>
     <plugin name="gazebo_ros_control" filename="libgazebo_ros_control.so">
-       <!--<robotNamespace>/shadowhand_motor</robotNamespace>-->
-      <!--<alwaysOn>true</alwaysOn>-->
-      <!--<updateRate>1400.0</updateRate>-->
-      <!-- <robotParam>sh_description</robotParam> -->
+      <!--<robotNamespace>/shadowhand_motor</robotNamespace>-->
+      <robotSimType>sr_gazebo_sim/SrGazeboHWSim</robotSimType>
     </plugin>
   </gazebo>
