Commit message: Remove contact sensors to avoid gazebo crash

File: sr_description/hand/xacro/finger/distal/distal.gazebo.xacro (robot description, xacro)
@@ -4,18 +4,4 @@
   <!-- prefix can be anything but usually is "r_" or  "l_" for right and left hands distinction -->
   <gazebo reference="${prefix}${link_prefix}distal">
-      <sensor type="contact" name="${prefix}${link_prefix}distal_contact">
-				<always_on>1</always_on>
-        <update_rate>1000.0</update_rate>
-        <contact>
-          <collision>${prefix}${link_prefix}distal_collision</collision>
-          <topic>${prefix}${link_prefix}distal_collision</topic>
-        </contact>
-        <plugin name="${prefix}${link_prefix}distal_gazebo_ros_bumper_controller" filename="libgazebo_ros_bumper.so">
-          <alwaysOn>true</alwaysOn>
-          <frameName>${prefix}${link_prefix}distal</frameName>
-          <updateRate>100.0</updateRate>
-          <bumperTopicName>contacts/${prefix}${link_prefix}/distal</bumperTopicName>
-        </plugin>
-      </sensor>
       <mu1 value="500.0" />
       <mu2 value="500.0" />

File: sr_description/hand/xacro/finger/knuckle/knuckle.gazebo.xacro (robot description, xacro)
@@ -4,18 +4,4 @@
   <!-- prefix can be anything but usually is "r_" or  "l_" for right and left hands distinction -->
   <gazebo reference="${prefix}${link_prefix}knuckle">
-      <sensor type="contact" name="${prefix}${link_prefix}knuckle_contact">
-				<always_on>1</always_on>
-        <update_rate>1000.0</update_rate>
-        <contact>
-          <collision>${prefix}${link_prefix}knuckle_collision</collision>
-          <topic>${prefix}${link_prefix}knuckle_collision</topic>
-        </contact>
-        <plugin name="${prefix}${link_prefix}knuckle_gazebo_ros_bumper_controller" filename="libgazebo_ros_bumper.so">
-          <alwaysOn>true</alwaysOn>
-          <frameName>${prefix}${link_prefix}knuckle</frameName>
-          <updateRate>100.0</updateRate>
-          <bumperTopicName>contacts/${prefix}${link_prefix}/knuckle</bumperTopicName>
-        </plugin>
-      </sensor>
       <material>Gazebo/Grey</material>
     </gazebo>

File: sr_description/hand/xacro/finger/lfmetacarpal/lfmetacarpal.gazebo.xacro (robot description, xacro)
@@ -4,18 +4,4 @@
   <!-- prefix can be anything but usually is "r_" or  "l_" for right and left hands distinction -->
   <gazebo reference="${prefix}lfmetacarpal">
-      <sensor type="contact" name="${prefix}lfmetacarpal_contact">
-				<always_on>1</always_on>
-        <update_rate>1000.0</update_rate>
-        <contact>
-          <collision>${prefix}lfmetacarpal_collision</collision>
-          <topic>${prefix}lfmetacarpal_collision</topic>
-        </contact>
-        <plugin name="${prefix}lfmetacarpal_gazebo_ros_bumper_controller" filename="libgazebo_ros_bumper.so">
-          <alwaysOn>true</alwaysOn>
-          <frameName>${prefix}lfmetacarpal</frameName>
-          <updateRate>100.0</updateRate>
-          <bumperTopicName>contacts/${prefix}lf/metacarpal</bumperTopicName>
-        </plugin>
-      </sensor>
       <selfCollide>true</selfCollide>
     </gazebo>

File: sr_description/hand/xacro/finger/middle/middle.gazebo.xacro (robot description, xacro)
@@ -4,18 +4,4 @@
   <!-- prefix can be anything but usually is "r_" or  "l_" for right and left hands distinction -->
   <gazebo reference="${prefix}${link_prefix}middle">
-      <sensor type="contact" name="${prefix}${link_prefix}middle_contact">
-        <always_on>1</always_on>
-        <update_rate>1000.0</update_rate>
-        <contact>
-          <collision>${prefix}${link_prefix}middle_collision</collision>
-          <topic>${prefix}${link_prefix}middle_collision</topic>
-        </contact>
-        <plugin name="${prefix}${link_prefix}proximal_gazebo_ros_bumper_controller" filename="libgazebo_ros_bumper.so">
-          <alwaysOn>true</alwaysOn>
-          <frameName>${prefix}${link_prefix}middle</frameName>
-          <updateRate>100.0</updateRate>
-          <bumperTopicName>contacts/${prefix}${link_prefix}/middle</bumperTopicName>
-        </plugin>
-      </sensor>
       <selfCollide>true</selfCollide>
     </gazebo>

File: sr_description/hand/xacro/finger/proximal/proximal.gazebo.xacro (robot description, xacro)
@@ -4,18 +4,4 @@
   <!-- prefix can be anything but usually is "r_" or  "l_" for right and left hands distinction -->
   <gazebo reference="${prefix}${link_prefix}proximal">
-      <sensor type="contact" name="${prefix}${link_prefix}proximal_contact">
-        <always_on>1</always_on>
-        <update_rate>1000.0</update_rate>
-        <contact>
-          <collision>${prefix}${link_prefix}proximal_collision</collision>
-          <topic>${prefix}${link_prefix}proximal_collision</topic>
-        </contact>
-        <plugin name="${prefix}${link_prefix}proximal_gazebo_ros_bumper_controller" filename="libgazebo_ros_bumper.so">
-          <alwaysOn>true</alwaysOn>
-          <frameName>${prefix}${link_prefix}proximal</frameName>
-          <updateRate>100.0</updateRate>
-          <bumperTopicName>contacts/${prefix}${link_prefix}/proximal</bumperTopicName>
-        </plugin>
-      </sensor>
       <selfCollide>true</selfCollide>
     </gazebo>

File: sr_description/hand/xacro/palm/palm.gazebo.xacro (robot description, xacro)
@@ -4,18 +4,4 @@
   <!-- prefix can be anything but usually is "r_" or  "l_" for right and left hands distinction -->
   <gazebo reference="${prefix}palm">
-      <sensor type="contact" name="${prefix}palm_contact">
-        <always_on>1</always_on>
-        <update_rate>1000.0</update_rate>
-        <contact>
-          <collision>${prefix}palm_collision</collision>
-          <topic>${prefix}palm_collision</topic>
-        </contact>
-        <plugin name="${prefix}palm_gazebo_ros_bumper_controller" filename="libgazebo_ros_bumper.so">
-          <alwaysOn>true</alwaysOn>
-          <frameName>${prefix}palm</frameName>
-          <updateRate>100.0</updateRate>
-          <bumperTopicName>contacts/${prefix}palm</bumperTopicName>
-        </plugin>
-      </sensor>
     </gazebo>
   </xacro:macro>

File: sr_description/hand/xacro/thumb/thbase.gazebo.xacro (robot description, xacro)
@@ -4,18 +4,4 @@
   <!-- prefix can be anything but usually is "r_" or  "l_" for right and left hands distinction -->
   <gazebo reference="${prefix}thbase">
-      <sensor type="contact" name="${prefix}thbase_contact">
-        <always_on>1</always_on>
-        <update_rate>1000.0</update_rate>
-        <contact>
-          <collision>${prefix}thbase_collision</collision>
-          <topic>${prefix}thbase_collision</topic>
-        </contact>
-        <plugin name="${prefix}thbase_gazebo_ros_bumper_controller" filename="libgazebo_ros_bumper.so">
-          <alwaysOn>true</alwaysOn>
-          <frameName>${prefix}thbase</frameName>
-          <updateRate>100.0</updateRate>
-          <bumperTopicName>contacts/${prefix}th/base</bumperTopicName>
-        </plugin>
-      </sensor>
       <selfCollide>false</selfCollide>
     </gazebo>

File: sr_description/hand/xacro/thumb/thdistal.gazebo.xacro (robot description, xacro)
@@ -4,18 +4,4 @@
   <!-- prefix can be anything but usually is "r_" or  "l_" for right and left hands distinction -->
   <gazebo reference="${prefix}thdistal">
-      <sensor type="contact" name="${prefix}thdistal_contact">
-        <always_on>1</always_on>
-        <update_rate>1000.0</update_rate>
-        <contact>
-          <collision>${prefix}thdistal_collision</collision>
-          <topic>${prefix}thdistal_collision</topic>
-        </contact>
-        <plugin name="${prefix}thdistal_gazebo_ros_bumper_controller" filename="libgazebo_ros_bumper.so">
-          <alwaysOn>true</alwaysOn>
-          <frameName>${prefix}thdistal</frameName>
-          <updateRate>100.0</updateRate>
-          <bumperTopicName>contacts/${prefix}th/distal</bumperTopicName>
-        </plugin>
-      </sensor>
       <mu1 value="500.0" />
       <mu2 value="500.0" />

File: sr_description/hand/xacro/thumb/thhub.gazebo.xacro (robot description, xacro)
@@ -4,18 +4,4 @@
   <!-- prefix can be anything but usually is "r_" or  "l_" for right and left hands distinction -->
   <gazebo reference="${prefix}thhub">
-      <sensor type="contact" name="${prefix}thhub_contact">
-        <always_on>1</always_on>
-        <update_rate>1000.0</update_rate>
-        <contact>
-          <collision>${prefix}thhub_collision</collision>
-          <topic>${prefix}thhub_collision</topic>
-        </contact>
-        <plugin name="${prefix}thhub_gazebo_ros_bumper_controller" filename="libgazebo_ros_bumper.so">
-          <alwaysOn>true</alwaysOn>
-          <frameName>${prefix}thhub</frameName>
-          <updateRate>100.0</updateRate>
-          <bumperTopicName>contacts/${prefix}th/hub</bumperTopicName>
-        </plugin>
-      </sensor>
       <selfCollide>true</selfCollide>
     </gazebo>

File: sr_description/hand/xacro/thumb/thmiddle.gazebo.xacro (robot description, xacro)
@@ -4,18 +4,4 @@
   <!-- prefix can be anything but usually is "r_" or  "l_" for right and left hands distinction -->
   <gazebo reference="${prefix}thmiddle">
-      <sensor type="contact" name="${prefix}thmiddle_contact">
-        <always_on>1</always_on>
-        <update_rate>1000.0</update_rate>
-        <contact>
-          <collision>${prefix}thmiddle_collision</collision>
-          <topic>${prefix}thmiddle_collision</topic>
-        </contact>
-        <plugin name="${prefix}thmiddle_gazebo_ros_bumper_controller" filename="libgazebo_ros_bumper.so">
-          <alwaysOn>true</alwaysOn>
-          <frameName>${prefix}thmiddle</frameName>
-          <updateRate>100.0</updateRate>
-          <bumperTopicName>contacts/${prefix}th/middle</bumperTopicName>
-        </plugin>
-      </sensor>
       <selfCollide>true</selfCollide>
     </gazebo>

File: sr_description/hand/xacro/thumb/thproximal.gazebo.xacro (robot description, xacro)
@@ -4,18 +4,4 @@
   <!-- prefix can be anything but usually is "r_" or  "l_" for right and left hands distinction -->
   <gazebo reference="${prefix}thproximal">
-      <sensor type="contact" name="${prefix}thproximal_contact">
-        <always_on>1</always_on>
-        <update_rate>1000.0</update_rate>
-        <contact>
-          <collision>${prefix}thproximal_collision</collision>
-          <topic>${prefix}thproximal_collision</topic>
-        </contact>
-        <plugin name="${prefix}thproximal_gazebo_ros_bumper_controller" filename="libgazebo_ros_bumper.so">
-          <alwaysOn>true</alwaysOn>
-          <frameName>${prefix}thproximal</frameName>
-          <updateRate>100.0</updateRate>
-          <bumperTopicName>contacts/${prefix}th/proximal</bumperTopicName>
-        </plugin>
-      </sensor>
       <selfCollide>false</selfCollide>
     </gazebo>

File: sr_description/other/xacro/gazebo/gazebo.urdf.xacro (robot description, xacro)
@@ -6,4 +6,5 @@
     <plugin name="gazebo_ros_control" filename="libgazebo_ros_control.so">
       <robotSimType>sr_gazebo_sim/SrGazeboHWSim</robotSimType>
+      <robotNamespace>sh</robotNamespace>
     </plugin>
   </gazebo>
